File: pcb/power.sch (KiCad schematic (older format))
At the start: 0 parts

Commit message: WIp battery controller
Changed lines of the file:
@@
 $Descr A4 11693 8268
 encoding utf-8
-Sheet 2 14
+Sheet 2 15
 Title "Power Supplies"
 Date ""
@@
 Text Notes 750  1250 0    118  ~ 24
 Power entry/battery stuff here etc. etc.
+$Sheet
+S 2400 3250 1550 750
+U 5FE1065D
+F0 "battery_controller" 50
+F1 "battery_controller.sch" 50
+$EndSheet
 $EndSCHEMATC
